Commit message: configurator + tool convention: visual port from robocore-studio (Inter / Tomorrow, teal accent on black, ghost buttons), preview-on-top responsive layout with Configuration + Joint pose on the right, dynamic joint sliders built from the loaded URDF, and a Home button that drives the arm to a defined ready pose   (joints 2/3/4 at -π/4, +π/2, -π/4) — matched by initial_value's in mod101.ros2control so Gazebo wakes up the same; adds docs/tool-convention.md and refactors parallel / pincopen / new mod101_tool_jaws onto it (each tool gets a _root link + identity mount + single _cad_to_root joint for CAD-frame conversion);   restores the original 136/140 mm extrusion lengths; paints the base cover, shoulder-elbow body, camera mount/tilter, elbow fork, and every tool body accent_green (Gazebo/Green in sim).

File: src/mod101_description/urdf/materials.xacro (robot description, xacro)
@@ -13,3 +13,8 @@
     <color rgba="0.700 0.700 0.700 1.0"/>
   </material>
+  <!-- Accent colour used on the base cover, the elbow_shoulder body, the elbow
+       fork, the camera mount/tilter, and every active tool's body links. -->
+  <material name="accent_green">
+    <color rgba="0.180 0.580 0.270 1.0"/>
+  </material>
 </robot>

File: src/mod101_description/urdf/mod101.xacro (robot description, xacro)
@@ -11,5 +11,5 @@
      its own launch fragment. Must match a package named
      `mod101_tool_<tool>` that ships urdf/tool.urdf.xacro. -->
-<xacro:arg name="tool" default="parallel"/>
+<xacro:arg name="tool" default="jaws"/>
 <xacro:include filename="$(find mod101_description)/urdf/materials.xacro" />
 <xacro:if value="$(arg use_sim)">
@@ -26,6 +26,6 @@
      The elbow link covers two parallel rails, so its mass is 2× density × L.
      ============================================================ -->
-<xacro:property name="shoulder_ext_length" value="0.0800"/>
-<xacro:property name="elbow_ext_length"    value="0.0800"/>
+<xacro:property name="shoulder_ext_length" value="0.1360"/>
+<xacro:property name="elbow_ext_length"    value="0.1400"/>
 <xacro:property name="extrusion_density"   value="0.46"/>
 <xacro:property name="ext_cross"           value="0.020"/>  <!-- 20x20 mm profile -->
@@ -91,5 +91,5 @@
       <mesh filename="file://$(find mod101_description)/meshes/base_cover_1.stl" scale="0.001 0.001 0.001"/>
     </geometry>
-    <material name="body_darkgrey"/>
+    <material name="accent_green"/>
   </visual>
   <collision>
@@ -430,5 +430,5 @@
       <mesh filename="file://$(find mod101_description)/meshes/shoulder_elbow_body_1.stl" scale="0.001 0.001 0.001"/>
     </geometry>
-    <material name="body_darkgrey"/>
+    <material name="accent_green"/>
   </visual>
   <collision>
@@ -450,5 +450,5 @@
       <mesh filename="file://$(find mod101_description)/meshes/camera_tilter_1.stl" scale="0.001 0.001 0.001"/>
     </geometry>
-    <material name="body_darkgrey"/>
+    <material name="accent_green"/>
   </visual>
   <collision>
@@ -470,5 +470,5 @@
       <mesh filename="file://$(find mod101_description)/meshes/camera_mount_1.stl" scale="0.001 0.001 0.001"/>
     </geometry>
-    <material name="body_darkgrey"/>
+    <material name="accent_green"/>
   </visual>
   <collision>
@@ -560,5 +560,5 @@
       <mesh filename="file://$(find mod101_description)/meshes/elbow_fork_1.stl" scale="0.001 0.001 0.001"/>
     </geometry>
-    <material name="body_darkgrey"/>
+    <material name="accent_green"/>
   </visual>
   <collision>
@@ -708,4 +708,7 @@
   <xacro:include filename="$(find mod101_tool_pincopen)/urdf/tool.urdf.xacro"/>
 </xacro:if>
+<xacro:if value="${'$(arg tool)' == 'jaws'}">
+  <xacro:include filename="$(find mod101_tool_jaws)/urdf/tool.urdf.xacro"/>
+</xacro:if>
 <xacro:if value="${'$(arg tool)' == 'none'}">
   <xacro:include filename="$(find mod101_tool_none)/urdf/tool.urdf.xacro"/>

File: src/mod101_tool_none/urdf/tool.urdf.xacro (robot description, xacro)
@@ -17,5 +17,5 @@
         <cylinder radius="0.025" length="0.010"/>
       </geometry>
-      <material name="body_darkgrey"/>
+      <material name="accent_green"/>
     </visual>
     <collision>
@@ -32,5 +32,5 @@
   </joint>
   <gazebo reference="end_cap">
-    <material>Gazebo/DarkGrey</material>
+    <material>Gazebo/Green</material>
     <mu1>0.2</mu1>
     <mu2>0.2</mu2>

File: src/mod101_tool_parallel/urdf/tool.urdf.xacro (robot description, xacro)
@@ -1,10 +1,37 @@
 <?xml version="1.0" ?>
 <!--
-  Parallel-jaw gripper tool. Mounts to the standard mod101 `wrist_flange`
-  contract: bolts on as a fixed child at the flange origin (Z out, X up).
+  Parallel-jaw gripper tool. Follows docs/tool-convention.md:
+    wrist_flange
+      └─[parallel_mount, identity]──> parallel_root
+           └─[parallel_cad_to_root, identity]──> Parallel_gripper_assembly_v1_1
+                 ├─[6, prismatic]──> left_jaw
+                 └─[right_jaw_slider, prismatic <mimic>]──> right_jaw
+  The vendored CAD sub-tree was authored such that its link origin already
+  coincides with the bolt pattern, so parallel_cad_to_root is identity —
+  parallel_root and Parallel_gripper_assembly_v1_1 are colocated.
 -->
 <robot xmlns:xacro="http://www.ros.org/wiki/xacro">
   <!-- ============================================================
-       Gripper body + jaws
+       Convention root: at the bolt pattern, +X outward, +Z up.
+       ============================================================ -->
+  <link name="parallel_root">
+    <inertial>
+      <origin xyz="0 0 0" rpy="0 0 0"/>
+      <mass value="0.001"/>
+      <inertia ixx="1e-7" iyy="1e-7" izz="1e-7" ixy="0" iyz="0" ixz="0"/>
+    </inertial>
+  </link>
+  <joint name="parallel_mount" type="fixed">
+    <origin xyz="0 0 0" rpy="0 0 0"/>
+    <parent link="wrist_flange"/>
+    <child  link="parallel_root"/>
+  </joint>
+  <joint name="parallel_cad_to_root" type="fixed">
+    <origin xyz="0 0 0" rpy="0 0 0"/>
+    <parent link="parallel_root"/>
+    <child  link="Parallel_gripper_assembly_v1_1"/>
+  </joint>
+  <!-- ============================================================
+       Gripper body + jaws (vendored CAD sub-tree)
        ============================================================ -->
   <link name="Parallel_gripper_assembly_v1_1">
@@ -19,5 +46,5 @@
         <mesh filename="package://mod101_tool_parallel/meshes/Parallel_gripper_assembly_v1_1.stl" scale="0.001 0.001 0.001"/>
       </geometry>
-      <material name="body_darkgrey"/>
+      <material name="accent_green"/>
     </visual>
     <collision>
@@ -39,5 +66,5 @@
         <mesh filename="package://mod101_tool_parallel/meshes/left_jaw_v1_1.stl" scale="0.001 0.001 0.001"/>
       </geometry>
-      <material name="body_darkgrey"/>
+      <material name="accent_green"/>
     </visual>
     <collision>
@@ -59,5 +86,5 @@
         <mesh filename="package://mod101_tool_parallel/meshes/right_jaw_v1_1.stl" scale="0.001 0.001 0.001"/>
       </geometry>
-      <material name="body_darkgrey"/>
+      <material name="accent_green"/>
     </visual>
     <collision>
@@ -71,10 +98,4 @@
        Joints
        ============================================================ -->
-  <!-- Fixed mount: gripper body bolts to the wrist flange contract. -->
-  <joint name="parallel_gripper_mount" type="fixed">
-    <origin xyz="0 0 0" rpy="0 0 0"/>
-    <parent link="wrist_flange"/>
-    <child link="Parallel_gripper_assembly_v1_1"/>
-  </joint>
   <joint name="6" type="prismatic">
     <origin xyz="0.04361 0.021616 0.020519" rpy="0 0 0"/>

File: src/mod101_tool_pincopen/urdf/tool.urdf.xacro (robot description, xacro)
@@ -9,6 +9,9 @@
     * single-active-joint design preserved: `6` is revolute, the four arm/
       finger joints follow via URDF <mimic> (works under bullet-featherstone).
-    * fixed-joint mount from `wrist_flange` -> `pincopen_base_link`. The
-      transform below is a placeholder — measure the adapter bracket and tune.
+    * mount layered per docs/tool-convention.md:
+        wrist_flange ─[pincopen_mount, identity]─> pincopen_root
+                     ─[pincopen_cad_to_root, identity]─> pincopen_base_link
+      (PincOpen's CAD frame already follows the convention so cad_to_root
+      is identity; tune that joint if reorientation becomes needed.)
     * minimal inertials added (upstream has none; gz_ros2_control needs them).
 -->
@@ -16,5 +19,30 @@
   <xacro:property name="mesh_scale" value="0.001 0.001 0.001"/>
   <!-- ============================================================
-       Links
+       Convention root: at the bolt pattern, +X outward, +Z up.
+       The vendored sub-tree starts at `pincopen_base_link`; PincOpen's CAD
+       frame happens to match the convention already (link origins coincide
+       with the wrist mount, mesh visual_origins are zero) so the
+       cad-to-root joint is identity. Tune rpy here if you need to reorient
+       the gripper.
+       ============================================================ -->
+  <link name="pincopen_root">
+    <inertial>
+      <origin xyz="0 0 0" rpy="0 0 0"/>
+      <mass value="0.001"/>
+      <inertia ixx="1e-7" iyy="1e-7" izz="1e-7" ixy="0" iyz="0" ixz="0"/>
+    </inertial>
+  </link>
+  <joint name="pincopen_mount" type="fixed">
+    <origin xyz="0 0 0" rpy="0 0 0"/>
+    <parent link="wrist_flange"/>
+    <child  link="pincopen_root"/>
+  </joint>
+  <joint name="pincopen_cad_to_root" type="fixed">
+    <origin xyz="0 0 0" rpy="0 0 0"/>
+    <parent link="pincopen_root"/>
+    <child  link="pincopen_base_link"/>
+  </joint>
+  <!-- ============================================================
+       Vendored PincOpen sub-tree
        ============================================================ -->
   <link name="pincopen_base_link">
@@ -29,5 +57,5 @@
         <mesh filename="package://mod101_tool_pincopen/meshes/Gripper_Palm_Shell_w_motor_v1.stl" scale="${mesh_scale}"/>
       </geometry>
-      <material name="body_darkgrey"/>
+      <material name="accent_green"/>
     </visual>
     <collision>
@@ -63,5 +91,5 @@
         <mesh filename="package://mod101_tool_pincopen/meshes/gripper_right_arm.stl" scale="${mesh_scale}"/>
       </geometry>
-      <material name="body_darkgrey"/>
+      <material name="accent_green"/>
     </visual>
     <collision>
@@ -83,5 +111,5 @@
         <mesh filename="package://mod101_tool_pincopen/meshes/gripper_left_arm.stl" scale="${mesh_scale}"/>
       </geometry>
-      <material name="body_darkgrey"/>
+      <material name="accent_green"/>
     </visual>
     <collision>
@@ -135,14 +163,4 @@
        Joints
        ============================================================ -->
-  <!-- Mount: gripper palm fixed to the wrist flange.
-       wrist_flange's +X is the wrist-roll axis = "outward" from the wrist.
-       PincOpen's local +X (from base_link toward the coupler at xyz=0.0535)
-       is the fingers-outward direction. Identity rpy aligns them so the
-       gripper projects straight out of the wrist with the motor on +Z. -->
-  <joint name="pincopen_mount" type="fixed">
-    <origin xyz="0 0 0" rpy="0 0 0"/>
-    <parent link="wrist_flange"/>
-    <child link="pincopen_base_link"/>
-  </joint>
   <!-- Single active joint. Named "6" to match the mod101 numbering. -->
   <joint name="6" type="revolute">
