Commit message: Part A: consolidate arm into one parametric URDF
Retrofit the modular mod101_arm macro with the integration spec's four build
args (shoulder_ext_length, elbow_ext_length, shoulder_mount, elbow_mount) so the
configurator drives any member of the family directly.

- Canonical joint vocabulary: joint_base / joint_shoulder / joint_elbow /
  joint_wrist_tilt / joint_wrist_roll; fixed joints -> fixed_<childlink>.
  No CAD auto-names remain (git grep -iE '(revolute|rigid) [0-9]' is clean).
- Elbow axis canonicalized to 0 1 0 (resolves the two exports' sign
  disagreement by construction). Base axis kept pending hardware confirmation.
- Per-joint mount selector (A3): big mount swaps servo body mass (56->105 g/half)
  and pushes the downstream joint axis out by a fixed delta (delta_shoulder,
  delta_elbow — provisional, FIXME for Cristi's CAD measurements).
- joint_wrist_roll stays actuated (A5 resolved: kept, drives the wrist_flange).
- Joint rename propagated to ros2control (sim + hardware) and controllers.yaml.
- CAD exports relocated to reference/ (untracked source geometry, not built).

Renders for all four mount combos; check_urdf parses the full robot.

Co-Authored-By: Claude Opus 4.8 (1M context) <noreply@anthropic.com>

File: src/mod101_control/urdf/mod101.hardware.xacro (robot description, xacro)
@@ -15,25 +15,25 @@
       <plugin>mock_components/GenericSystem</plugin>
     </hardware>
-    <joint name="1">
+    <joint name="joint_base">
       <command_interface name="position"/>
       <state_interface name="position"/>
       <state_interface name="velocity"/>
     </joint>
-    <joint name="2">
+    <joint name="joint_shoulder">
       <command_interface name="position"/>
       <state_interface name="position"/>
       <state_interface name="velocity"/>
     </joint>
-    <joint name="3">
+    <joint name="joint_elbow">
       <command_interface name="position"/>
       <state_interface name="position"/>
       <state_interface name="velocity"/>
     </joint>
-    <joint name="4">
+    <joint name="joint_wrist_tilt">
       <command_interface name="position"/>
       <state_interface name="position"/>
       <state_interface name="velocity"/>
     </joint>
-    <joint name="5">
+    <joint name="joint_wrist_roll">
       <command_interface name="position"/>
       <state_interface name="position"/>

File: src/mod101_description/urdf/mod101.xacro (robot description, xacro)
@@ -1,3 +1,10 @@
 <?xml version="1.0" ?>
+<!--
+  Standalone mod101 entry point: one arm anchored to the world. The arm
+  itself lives in mod101_macro.xacro as the prefix-parameterised
+  `mod101_arm` macro so other robots (e.g. base101's dual-arm tower) can
+  instantiate it any number of times — include that file directly, not
+  this one.
+-->
 <robot name="mod101" xmlns:xacro="http://www.ros.org/wiki/xacro">
 <!-- use_sim: when true, pulls in the Gazebo ros2_control system + per-link
@@ -12,705 +19,46 @@
      `mod101_tool_<tool>` that ships urdf/tool.urdf.xacro. -->
 <xacro:arg name="tool" default="jaws"/>
+<!-- Build parameters (the configurator's four inputs). These resolve any
+     member of the mod101 family: two rail lengths + two servo-mount variants.
+       *_ext_length  upper-arm / forearm 2020 rail length, m (configurator: the
+                     two length sliders; STS3215/3250 motor dropdown -> small,
+                     ST3120 -> big).
+       *_mount       'small' (STS3215/3250) | 'big' (ST3120). -->
+<xacro:arg name="shoulder_ext_length" default="0.1360"/>
+<xacro:arg name="elbow_ext_length"    default="0.1400"/>
+<xacro:arg name="shoulder_mount"      default="small"/>
+<xacro:arg name="elbow_mount"         default="small"/>
 <xacro:include filename="$(find mod101_description)/urdf/materials.xacro" />
-<xacro:if value="$(arg use_sim)">
-  <xacro:include filename="$(find mod101_description)/urdf/mod101.ros2control" />
-  <xacro:include filename="$(find mod101_description)/urdf/mod101.gazebo" />
-</xacro:if>
-<!-- ============================================================
-     Configurable 2020 aluminum extrusion lengths.
-     The web app edits ONLY these two property values; every dependent
-     quantity (joint offsets, box visuals, masses, inertias) recomputes.
-       shoulder_ext_length  - upper-arm rails (L and R, single 2020 each)
-       elbow_ext_length     - forearm dual-rail segment (one URDF link)
-     extrusion_density is the linear mass of one 2020 rail (kg/m).
-     The elbow link covers two parallel rails, so its mass is 2× density × L.
-     ============================================================ -->
-<xacro:property name="shoulder_ext_length" value="0.1360"/>
-<xacro:property name="elbow_ext_length"    value="0.1400"/>
-<xacro:property name="extrusion_density"   value="0.46"/>
-<xacro:property name="ext_cross"           value="0.020"/>  <!-- 20x20 mm profile -->
-<xacro:property name="ext_angle"           value="${pi/4}"/> <!-- both rails mount at 45 deg -->
-<xacro:property name="cos_a"               value="${cos(ext_angle)}"/>
-<xacro:property name="sin_a"               value="${sin(ext_angle)}"/>
+<xacro:include filename="$(find mod101_description)/urdf/mod101_macro.xacro" />
 <!-- Anchor base_link to the world so the arm doesn't tip over under gravity. -->
 <link name="world"/>
-<joint name="world_to_base" type="fixed">
-  <parent link="world"/>
-  <child link="base_link"/>
-  <origin xyz="0 0 0" rpy="0 0 0"/>
-</joint>
-<link name="base_link">
-  <inertial>
-    <origin xyz="-0.01099401981130007 1.3821647392049386e-05 0.013450739285809572" rpy="0 0 0"/>
-    <mass value="0.03628"/>
-    <inertia ixx="3.23936e-05" iyy="2.73718e-05" izz="4.10577e-05" ixy="0.0" iyz="0.0" ixz="5.68406e-06"/>
-  </inertial>
-  <visual>
-    <origin xyz="0 0 0" rpy="0 0 0"/>
-    <geometry>
-      <mesh filename="file://$(find mod101_description)/meshes/base_link.stl" scale="0.001 0.001 0.001"/>
-    </geometry>
-    <material name="body_darkgrey"/>
-  </visual>
-  <collision>
-    <origin xyz="0 0 0" rpy="0 0 0"/>
-    <geometry>
-      <mesh filename="file://$(find mod101_description)/meshes/base_link.stl" scale="0.001 0.001 0.001"/>
-    </geometry>
-  </collision>
-</link>
-<link name="servo_base_rotation_1">
-  <inertial>
-    <origin xyz="0.016199027563209848 0.010250000006755487 -0.015772935075263637" rpy="0 0 0"/>
-    <mass value="0.056"/>
-    <inertia ixx="7.87891e-06" iyy="1.4379e-05" izz="1.22123e-05" ixy="0.0" iyz="0.0" ixz="-1.96973e-07"/>
-  </inertial>
-  <visual>
-    <origin xyz="0.0166 0.01025 -0.05" rpy="0 0 0"/>
-    <geometry>
-      <mesh filename="file://$(find mod101_description)/meshes/servo_base_rotation_1.stl" scale="0.001 0.001 0.001"/>
-    </geometry>
-    <material name="motor_black"/>
-  </visual>
-  <collision>
-    <origin xyz="0.0166 0.01025 -0.05" rpy="0 0 0"/>
-    <geometry>
-      <mesh filename="file://$(find mod101_description)/meshes/servo_base_rotation_1.stl" scale="0.001 0.001 0.001"/>
-    </geometry>
-  </collision>
-</link>
-<link name="base_cover_1">
-  <inertial>
-    <origin xyz="0.02230032288194256 0.015943258220063473 1.6681447889688172e-12" rpy="0 0 0"/>
-    <mass value="0.01496"/>
-    <inertia ixx="4.77098e-06" iyy="8.58776e-06" izz="1.12913e-05" ixy="7.95163e-08" iyz="0.0" ixz="0.0"/>
-  </inertial>
-  <visual>
-    <origin xyz="0.028504 0.01555 -0.0338" rpy="0 0 0"/>
-    <geometry>
-      <mesh filename="file://$(find mod101_description)/meshes/base_cover_1.stl" scale="0.001 0.001 0.001"/>
-    </geometry>
-    <material name="accent_green"/>
-  </visual>
-  <collision>
-    <origin xyz="0.028504 0.01555 -0.0338" rpy="0 0 0"/>
-    <geometry>
-      <mesh filename="file://$(find mod101_description)/meshes/base_cover_1.stl" scale="0.001 0.001 0.001"/>
-    </geometry>
-  </collision>
-</link>
-<link name="base_rotation_body_1">
-  <inertial>
-    <origin xyz="0.035322745794806994 1.0118106741288103e-05 -0.025518978505968827" rpy="0 0 0"/>
-    <mass value="0.03606"/>
-    <inertia ixx="2.57397e-05" iyy="1.20767e-05" izz="2.58421e-05" ixy="0.0" iyz="0.0" ixz="3.07034e-07"/>
-  </inertial>
-  <visual>
-    <origin xyz="-0.0124 -0.0 -0.0528" rpy="0 0 0"/>
-    <geometry>
-      <mesh filename="file://$(find mod101_description)/meshes/base_rotation_body_1.stl" scale="0.001 0.001 0.001"/>
-    </geometry>
-    <material name="body_darkgrey"/>
-  </visual>
-  <collision>
-    <origin xyz="-0.0124 -0.0 -0.0528" rpy="0 0 0"/>
-    <geometry>
-      <mesh filename="file://$(find mod101_description)/meshes/base_rotation_body_1.stl" scale="0.001 0.001 0.001"/>
-    </geometry>
-  </collision>
-</link>
-<link name="servo_elbow_L_1">
-  <inertial>
-    <origin xyz="0.021389115640943528 -0.016027534864448984 0.006893671638235566" rpy="0 0 0"/>
-    <mass value="0.056"/>
-    <inertia ixx="1.12274e-05" iyy="1.22123e-05" izz="1.12274e-05" ixy="0.0" iyz="0.0" ixz="-3.34854e-06"/>
-  </inertial>
-  <visual>
-    <origin xyz="0.080166 -0.038392 -0.213311" rpy="0 0 0"/>
-    <geometry>
-      <mesh filename="file://$(find mod101_description)/meshes/servo_elbow_L_1.stl" scale="0.001 0.001 0.001"/>
-    </geometry>
-    <material name="motor_black"/>
-  </visual>
-  <collision>
-    <origin xyz="0.080166 -0.038392 -0.213311" rpy="0 0 0"/>
-    <geometry>
-      <mesh filename="file://$(find mod101_description)/meshes/servo_elbow_L_1.stl" scale="0.001 0.001 0.001"/>
-    </geometry>
-  </collision>
-</link>
-<!-- Elbow extrusion: dual 2020 rail (single URDF link representing both).
-     Geometry derives from elbow_ext_length and the fixed +45 deg mount angle. -->
-<link name="elbow_extrusion_1">
-  <xacro:property name="L" value="${elbow_ext_length}"/>
-  <xacro:property name="m" value="${2 * extrusion_density * L}"/>
-  <inertial>
-    <origin xyz="${L/2*cos_a} 0 ${L/2*sin_a}" rpy="0 ${ext_angle} 0"/>
-    <mass value="${m}"/>
-    <inertia ixx="${m*(ext_cross*ext_cross + L*L)/12}"
-             iyy="${m*(ext_cross*ext_cross + L*L)/12}"
-             izz="${m*(ext_cross*ext_cross + ext_cross*ext_cross)/12}"
-             ixy="0" iyz="0" ixz="0"/>
-  </inertial>
-  <visual>
-    <origin xyz="${L/2*cos_a} 0 ${L/2*sin_a}" rpy="0 ${ext_angle} 0"/>
-    <geometry>
-      <box size="${ext_cross} ${ext_cross} ${L}"/>
-    </geometry>
-    <material name="silver"/>
-  </visual>
-  <collision>
-    <origin xyz="${L/2*cos_a} 0 ${L/2*sin_a}" rpy="0 ${ext_angle} 0"/>
-    <geometry>
-      <box size="${ext_cross} ${ext_cross} ${L}"/>
-    </geometry>
-  </collision>
-</link>
-<link name="elbow_wrist_body_1">
-  <inertial>
-    <origin xyz="-0.0016612281041332028 0.00030497152583617594 -0.0016596828945049658" rpy="0 0 0"/>
-    <mass value="0.01"/>
-    <inertia ixx="2.37186e-06" iyy="1.25181e-06" izz="2.37186e-06" ixy="0.0" iyz="0.0" ixz="1.3177e-07"/>
-  </inertial>
-  <visual>
-    <origin xyz="-0.067372 0.000108 -0.346353" rpy="0 0 0"/>
-    <geometry>
-      <mesh filename="file://$(find mod101_description)/meshes/elbow_wrist_body_1.stl" scale="0.001 0.001 0.001"/>
-    </geometry>
-    <material name="body_darkgrey"/>
-  </visual>
-  <collision>
-    <origin xyz="-0.067372 0.000108 -0.346353" rpy="0 0 0"/>
-    <geometry>
-      <mesh filename="file://$(find mod101_description)/meshes/elbow_wrist_body_1.stl" scale="0.001 0.001 0.001"/>
-    </geometry>
-  </collision>
-</link>
-<link name="servo_wrist_tilt_1">
-  <inertial>
-    <origin xyz="0.018702326137297595 -0.015773405015014702 0.004206882115486588" rpy="0 0 0"/>
-    <mass value="0.056"/>
-    <inertia ixx="1.12274e-05" iyy="1.22123e-05" izz="1.12274e-05" ixy="0.0" iyz="0.0" ixz="-3.34854e-06"/>
-  </inertial>
-  <visual>
-    <origin xyz="-0.069599 -0.015892 -0.363076" rpy="0 0 0"/>
-    <geometry>
-      <mesh filename="file://$(find mod101_description)/meshes/servo_wrist_tilt_1.stl" scale="0.001 0.001 0.001"/>
-    </geometry>
-    <material name="motor_black"/>
-  </visual>
-  <collision>
-    <origin xyz="-0.069599 -0.015892 -0.363076" rpy="0 0 0"/>
-    <geometry>
-      <mesh filename="file://$(find mod101_description)/meshes/servo_wrist_tilt_1.stl" scale="0.001 0.001 0.001"/>
-    </geometry>
-  </collision>
-</link>
-<link name="wrist_tilt_body_1">
-  <inertial>
-    <origin xyz="0.02524119619320095 -0.018651053893336624 0.01828846906369841" rpy="0 0 0"/>
-    <mass value="0.01421"/>
-    <inertia ixx="8.22636e-06" iyy="9.3232e-06" izz="6.34605e-06" ixy="0.0" iyz="0.0" ixz="-3.2122e-06"/>
-  </inertial>
-  <visual>
-    <origin xyz="-0.097353 -0.018592 -0.376335" rpy="0 0 0"/>
-    <geometry>
-      <mesh filename="file://$(find mod101_description)/meshes/wrist_tilt_body_1.stl" scale="0.001 0.001 0.001"/>
-    </geometry>
-    <material name="body_darkgrey"/>
-  </visual>
-  <collision>
-    <origin xyz="-0.097353 -0.018592 -0.376335" rpy="0 0 0"/>
-    <geometry>
-      <mesh filename="file://$(find mod101_description)/meshes/wrist_tilt_body_1.stl" scale="0.001 0.001 0.001"/>
-    </geometry>
-  </collision>
-</link>
-<link name="servo_base_rotation__1__1">
-  <inertial>
-    <origin xyz="0.016027045473077706 0.010249530067015771 -0.019999491027092475" rpy="0 0 0"/>
-    <mass value="0.056"/>
-    <inertia ixx="1.22123e-05" iyy="1.4379e-05" izz="7.87891e-06" ixy="0.0" iyz="0.0" ixz="1.96973e-07"/>
-  </inertial>
-  <visual>
-    <origin xyz="-0.124753 0.010308 -0.409085" rpy="0 0 0"/>
-    <geometry>
-      <mesh filename="file://$(find mod101_description)/meshes/servo_base_rotation__1__1.stl" scale="0.001 0.001 0.001"/>
-    </geometry>
-    <material name="motor_black"/>
-  </visual>
-  <collision>
-    <origin xyz="-0.124753 0.010308 -0.409085" rpy="0 0 0"/>
-    <geometry>
-      <mesh filename="file://$(find mod101_description)/meshes/servo_base_rotation__1__1.stl" scale="0.001 0.001 0.001"/>
-    </geometry>
-  </collision>
-</link>
-<link name="shoulder_thingy_R_1">
-  <inertial>
-    <origin xyz="-8.767897172190509e-10 0.012838206577361115 0.004551181846450855" rpy="0 0 0"/>
-    <mass value="0.005"/>
-    <inertia ixx="8.39431e-07" iyy="3.49763e-07" izz="1.11924e-06" ixy="0.0" iyz="0.0" ixz="0.0"/>
-  </inertial>
-  <visual>
-    <origin xyz="-0.0504 0.035245 -0.0346" rpy="0 0 0"/>
-    <geometry>
-      <mesh filename="file://$(find mod101_description)/meshes/shoulder_thingy_R_1.stl" scale="0.001 0.001 0.001"/>
-    </geometry>
-    <material name="body_darkgrey"/>
-  </visual>
-  <collision>
-    <origin xyz="-0.0504 0.035245 -0.0346" rpy="0 0 0"/>
-    <geometry>
-      <mesh filename="file://$(find mod101_description)/meshes/shoulder_thingy_R_1.stl" scale="0.001 0.001 0.001"/>
-    </geometry>
-  </collision>
-</link>
-<link name="shoulder_thingy_L_1">
-  <inertial>
-    <origin xyz="-9.9631208838602e-10 -0.012838206577359481 0.004551181846451098" rpy="0 0 0"/>
-    <mass value="0.005"/>
-    <inertia ixx="8.39431e-07" iyy="3.49763e-07" izz="1.11924e-06" ixy="0.0" iyz="0.0" ixz="0.0"/>
-  </inertial>
-  <visual>
-    <origin xyz="-0.0504 -0.035245 -0.0346" rpy="0 0 0"/>
-    <geometry>
-      <mesh filename="file://$(find mod101_description)/meshes/shoulder_thingy_L_1.stl" scale="0.001 0.001 0.001"/>
-    </geometry>
-    <material name="body_darkgrey"/>
-  </visual>
-  <collision>
-    <origin xyz="-0.0504 -0.035245 -0.0346" rpy="0 0 0"/>
-    <geometry>
-      <mesh filename="file://$(find mod101_description)/meshes/shoulder_thingy_L_1.stl" scale="0.001 0.001 0.001"/>
-    </geometry>
-  </collision>
-</link>
-<link name="servo_shoulder_L_1">
-  <inertial>
-    <origin xyz="-0.010250001879856738 0.01577339742512835 0.01619857022441154" rpy="0 0 0"/>
-    <mass value="0.056"/>
-    <inertia ixx="1.4379e-05" iyy="1.22123e-05" izz="7.87891e-06" ixy="0.0" iyz="1.96973e-07" ixz="0.0"/>
-  </inertial>
-  <visual>
-    <origin xyz="-0.06065 -0.006247 -0.048652" rpy="0 0 0"/>
-    <geometry>
-      <mesh filename="file://$(find mod101_description)/meshes/servo_shoulder_L_1.stl" scale="0.001 0.001 0.001"/>
-    </geometry>
-    <material name="motor_black"/>
-  </visual>
-  <collision>
-    <origin xyz="-0.06065 -0.006247 -0.048652" rpy="0 0 0"/>
-    <geometry>
-      <mesh filename="file://$(find mod101_description)/meshes/servo_shoulder_L_1.stl" scale="0.001 0.001 0.001"/>
-    </geometry>
-  </collision>
-</link>
-<link name="servo_shoulder_R_1">
-  <inertial>
-    <origin xyz="-0.010249999993244191 0.016026997214310577 0.019998570224410886" rpy="0 0 0"/>
-    <mass value="0.056"/>
-    <inertia ixx="1.4379e-05" iyy="1.22123e-05" izz="7.87891e-06" ixy="0.0" iyz="-1.96973e-07" ixz="0.0"/>
-  </inertial>
-  <visual>
-    <origin xyz="-0.06065 0.038244 -0.044902" rpy="0 0 0"/>
-    <geometry>
-      <mesh filename="file://$(find mod101_description)/meshes/servo_shoulder_R_1.stl" scale="0.001 0.001 0.001"/>
-    </geometry>
-    <material name="motor_black"/>
-  </visual>
-  <collision>
-    <origin xyz="-0.06065 0.038244 -0.044902" rpy="0 0 0"/>
-    <geometry>
-      <mesh filename="file://$(find mod101_description)/meshes/servo_shoulder_R_1.stl" scale="0.001 0.001 0.001"/>
-    </geometry>
-  </collision>
-</link>
-<link name="shoulder_fork_1">
-  <inertial>
-    <origin xyz="-0.017328700920341188 -0.04029953765013844 0.017328241708440162" rpy="0 0 0"/>
-    <mass value="0.022"/>
-    <inertia ixx="1.78124e-05" iyy="4.46929e-06" izz="1.78124e-05" ixy="0.0" iyz="0.0" ixz="9.71586e-07"/>
-  </inertial>
-  <visual>
-    <origin xyz="-0.0504 -0.040447 -0.077652" rpy="0 0 0"/>
-    <geometry>
-      <mesh filename="file://$(find mod101_description)/meshes/shoulder_fork_1.stl" scale="0.001 0.001 0.001"/>
-    </geometry>
-    <material name="body_darkgrey"/>
-  </visual>
-  <collision>
-    <origin xyz="-0.0504 -0.040447 -0.077652" rpy="0 0 0"/>
-    <geometry>
-      <mesh filename="file://$(find mod101_description)/meshes/shoulder_fork_1.stl" scale="0.001 0.001 0.001"/>
-    </geometry>
-  </collision>
-</link>
-<!-- Shoulder extrusions: two parallel single 2020 rails, modeled as separate
-     URDF links. Rail direction (-1, 0, 1)/sqrt(2) in each rail's local frame. -->
-<link name="shoulder_extrusion_R_1">
-  <xacro:property name="L" value="${shoulder_ext_length}"/>
-  <xacro:property name="m" value="${extrusion_density * L}"/>
-  <inertial>
-    <origin xyz="${-L/2*cos_a} 0 ${L/2*sin_a}" rpy="0 ${-ext_angle} 0"/>
-    <mass value="${m}"/>
-    <inertia ixx="${m*(ext_cross*ext_cross + L*L)/12}"
-             iyy="${m*(ext_cross*ext_cross + L*L)/12}"
-             izz="${m*(ext_cross*ext_cross + ext_cross*ext_cross)/12}"
-             ixy="0" iyz="0" ixz="0"/>
-  </inertial>
-  <visual>
-    <origin xyz="${-L/2*cos_a} 0 ${L/2*sin_a}" rpy="0 ${-ext_angle} 0"/>
-    <geometry>
-      <box size="${ext_cross} ${ext_cross} ${L}"/>
-    </geometry>
-    <material name="silver"/>
-  </visual>
-  <collision>
-    <origin xyz="${-L/2*cos_a} 0 ${L/2*sin_a}" rpy="0 ${-ext_angle} 0"/>
-    <geometry>
-      <box size="${ext_cross} ${ext_cross} ${L}"/>
-    </geometry>
-  </collision>
-</link>
-<link name="shoulder_extrusion_L_1">
-  <xacro:property name="L" value="${shoulder_ext_length}"/>
-  <xacro:property name="m" value="${extrusion_density * L}"/>
-  <inertial>
-    <origin xyz="${-L/2*cos_a} 0 ${L/2*sin_a}" rpy="0 ${-ext_angle} 0"/>
-    <mass value="${m}"/>
-    <inertia ixx="${m*(ext_cross*ext_cross + L*L)/12}"
-             iyy="${m*(ext_cross*ext_cross + L*L)/12}"
-             izz="${m*(ext_cross*ext_cross + ext_cross*ext_cross)/12}"
-             ixy="0" iyz="0" ixz="0"/>
-  </inertial>
-  <visual>
-    <origin xyz="${-L/2*cos_a} 0 ${L/2*sin_a}" rpy="0 ${-ext_angle} 0"/>
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