Commit message: big changes

File: src/mod101_control/urdf/mod101.hardware.xacro (robot description, xacro)
@@ -35,4 +35,14 @@
       <state_interface name="velocity"/>
     </joint>
+    <joint name="joint_wrist_roll">
+      <command_interface name="position"/>
+      <state_interface name="position"/>
+      <state_interface name="velocity"/>
+    </joint>
+    <!-- No tool joint here on purpose. Each mod101_tool_* package emits its own
+         <ros2_control> block (urdf/tool.ros2control) in BOTH sim and hardware
+         modes, already declaring its `6` joint with the right limits. Declaring
+         it here too would have two hardware components claiming one joint,
+         which controller_manager rejects at load. -->
   </ros2_control>
 </robot>

File: src/mod101_description/urdf/mod101.xacro (robot description, xacro)
@@ -5,6 +5,6 @@
   other robots can instantiate it any number of times — include that file
   directly, not this one.
-  Tools and the configurator are handled separately (later). This standalone is
-  the bare arm, drivable in Gazebo via ros2_control.
+  Drivable in Gazebo via ros2_control, with the end-effector selected by the
+  `tool` arg.
 -->
 <robot name="mod101" xmlns:xacro="http://www.ros.org/wiki/xacro">
@@ -12,4 +12,11 @@
      gazebo extensions. Hardware overlays (mod101_control) override to false. -->
 <xacro:arg name="use_sim" default="true"/>
+<!-- tool: which end-effector package to pull in. The arm terminates at
+     `wrist_flange`; the selected tool's URDF attaches its root link there and
+     contributes its own joints, ros2_control hardware block, gazebo extensions,
+     controllers, and (via the gazebo launch) its own launch fragment. Must
+     match a package `mod101_tool_<tool>` shipping urdf/tool.urdf.xacro.
+     The configurator reads/writes this default. -->
+<xacro:arg name="tool" default="pincopen"/>
 <!-- Build parameters: two rail lengths + two servo-mount variants (small|big). -->
 <xacro:arg name="shoulder_ext_length" default="0.0820"/>
@@ -21,14 +28,29 @@
 <!-- Anchor base_link to the world so the arm doesn't tip over under gravity. -->
 <link name="world"/>
-<xacro:mod101_arm prefix="" parent="world" use_sim="$(arg use_sim)"
+<xacro:mod101_arm prefix="" parent="world" tool="$(arg tool)" use_sim="$(arg use_sim)"
                   shoulder_ext_length="$(arg shoulder_ext_length)"
                   elbow_ext_length="$(arg elbow_ext_length)"
                   shoulder_mount="$(arg shoulder_mount)"
                   elbow_mount="$(arg elbow_mount)"/>
-<!-- gz_ros2_control plugin: exactly once per robot. Loads the arm controllers. -->
+<!-- gz_ros2_control plugin: exactly once per robot, so it lives here rather than
+     in the macro. It loads BOTH the arm's controller yaml and the active tool's
+     — gz_ros2_control merges multiple <parameters> files into the model's single
+     controller_manager namespace, so a tool contributes controllers without
+     touching this file. Integrators with their own plugin declaration (e.g.
+     base101) use the macro directly and skip this block. -->
 <xacro:if value="$(arg use_sim)">
   <gazebo>
     <plugin filename="gz_ros2_control-system" name="gz_ros2_control::GazeboSimROS2ControlPlugin">
       <parameters>$(find mod101_control)/config/controllers.sim.yaml</parameters>
+      <!-- Tool-specific controllers yaml. mod101_tool_none ships none. -->
+      <xacro:if value="${'$(arg tool)' == 'parallel'}">
+        <parameters>$(find mod101_tool_parallel)/config/controllers.yaml</parameters>
+      </xacro:if>
+      <xacro:if value="${'$(arg tool)' == 'pincopen'}">
+        <parameters>$(find mod101_tool_pincopen)/config/controllers.yaml</parameters>
+      </xacro:if>
+      <xacro:if value="${'$(arg tool)' == 'jaws'}">
+        <parameters>$(find mod101_tool_jaws)/config/controllers.yaml</parameters>
+      </xacro:if>
     </plugin>
   </gazebo>

File: src/mod101_description/urdf/mod101_macro.xacro (robot description, xacro)
@@ -12,9 +12,10 @@
                                              (mesh + mass). Everything else is
                                              identical between the two exports.
-  Tools and the configurator are handled separately (later); this macro is the
-  bare arm, testable in Gazebo with ros2_control.
+  The arm terminates at ${prefix}wrist_flange; the tool selected by the `tool`
+  param bolts its root link there (see docs/tool-convention.md).
   prefix   prepended to every link/joint name (multiple instances coexist).
   parent   link to bolt the base onto via a fixed ${prefix}base_mount joint.
            Empty = caller anchors ${prefix}base_link (mod101.xacro does).
+  tool     end-effector package suffix (mod101_tool_<tool>).
   use_sim  emit the gz_ros2_control hardware block + gazebo extensions.
 -->
@@ -22,4 +23,10 @@
 <xacro:include filename="$(find mod101_description)/urdf/mod101.ros2control"/>
 <xacro:include filename="$(find mod101_description)/urdf/mod101.gazebo"/>
+<!-- Every tool macro is included unconditionally (xacro has no conditional
+     include); only the one selected by `tool` is instantiated below. -->
+<xacro:include filename="$(find mod101_tool_parallel)/urdf/tool.urdf.xacro"/>
+<xacro:include filename="$(find mod101_tool_pincopen)/urdf/tool.urdf.xacro"/>
+<xacro:include filename="$(find mod101_tool_jaws)/urdf/tool.urdf.xacro"/>
+<xacro:include filename="$(find mod101_tool_none)/urdf/tool.urdf.xacro"/>
 <!-- Swappable joint modules (shoulder/elbow, small/big). Same pattern as the
      tools: each module is a self-contained sub-tree (prev link + servo + next
@@ -34,5 +41,5 @@
 <xacro:property name="ext_cross"         value="0.020"/>  <!-- 20x20 mm -->
 <xacro:property name="extrusion_density" value="0.46"/>   <!-- kg/m -->
-<xacro:macro name="mod101_arm" params="prefix:='' parent:='' xyz:='0 0 0' rpy:='0 0 0' use_sim:='true' shoulder_ext_length:='0.082' elbow_ext_length:='0.098' shoulder_mount:='small' elbow_mount:='small'">
+<xacro:macro name="mod101_arm" params="prefix:='' parent:='' xyz:='0 0 0' rpy:='0 0 0' tool:='jaws' use_sim:='true' shoulder_ext_length:='0.082' elbow_ext_length:='0.098' shoulder_mount:='small' elbow_mount:='small'">
 <!-- Rail length IS the joint advance along local X (1:1). The extrusion link is
      a box primitive of this length, so editing the length scales the rail AND
@@ -272,4 +279,14 @@
   </collision>
 </link>
+<!-- Wrist flange: the mount contract for tool packages (docs/tool-convention.md).
+     Massless frame on the wrist-roll servo's output horn; the active tool bolts
+     its root link here with an identity fixed joint. +X outward, +Z up. -->
+<link name="${prefix}wrist_flange">
+  <inertial>
+    <origin xyz="0 0 0" rpy="0 0 0"/>
+    <mass value="0.001"/>
+    <inertia ixx="1e-06" iyy="1e-06" izz="1e-06" ixy="0" iyz="0" ixz="0"/>
+  </inertial>
+</link>
 <!-- ===================== joints (canonical names, export axes) ============== -->
 <joint name="${prefix}fixed_servo_base_1" type="fixed">
@@ -336,4 +353,25 @@
   <child link="${prefix}servo_wrist_rotation_1"/>
 </joint>
+<!-- joint_wrist_roll: the actuated 5th DOF. The servo BODY is fixed to the
+     wrist_roll_adapter above; this joint is its output horn, driving the
+     wrist_flange (and hence the tool).
+     Origin/axis are derived from the export's own servo geometry rather than
+     measured separately: servo_wrist_rotation_1 is the same STS3215 part as
+     servo_base_1, rotated +90 deg about Y. Its inertia tensor is servo_base_1's
+     with ixx/izz swapped, and its COM is servo_base_1's COM under
+     (x,y,z) -> (z,y,-x) — both confirm that rotation exactly. Applying the same
+     map to joint_base's output (0.029, -0.01025, 0.0032) about axis +Z gives
+     the values below, about axis +X. +X is outward, per docs/tool-convention.md.
+     The flange sits ON the horn face: any adapter/spacer plate belongs to the
+     tool package, not here (tool-convention.md, "What this means for the mount
+     joint"). FIXME: confirm against CAD if a flange plate is ever added. -->
+<joint name="${prefix}joint_wrist_roll" type="continuous">
+  <origin xyz="0.0032 -0.01025 -0.029" rpy="0 0 0"/>
+  <parent link="${prefix}servo_wrist_rotation_1"/>
+  <child link="${prefix}wrist_flange"/>
+  <axis xyz="1.0 0.0 0.0"/>
+  <limit effort="100" velocity="100"/>
+  <dynamics damping="${joint_damping}" friction="${joint_friction}"/>
+</joint>
 <joint name="${prefix}fixed_camera_adapter_1" type="fixed">
   <origin xyz="0.0574 0.02935 0.0464" rpy="0 0 0"/>
@@ -355,4 +393,20 @@
   <xacro:mod101_arm_gazebo prefix="${prefix}"/>
 </xacro:if>
+<!-- Active end-effector. Each tool macro bolts its root link to wrist_flange
+     and contributes its own joints, ros2_control block and gazebo extensions.
+     Its controllers come from mod101.xacro's plugin block; its runtime nodes
+     from mod101_tool_<tool>/launch/tool.launch.py. -->
+<xacro:if value="${tool == 'parallel'}">
+  <xacro:mod101_tool_parallel prefix="${prefix}" use_sim="${use_sim}"/>
+</xacro:if>
+<xacro:if value="${tool == 'pincopen'}">
+  <xacro:mod101_tool_pincopen prefix="${prefix}" use_sim="${use_sim}"/>
+</xacro:if>
+<xacro:if value="${tool == 'jaws'}">
+  <xacro:mod101_tool_jaws prefix="${prefix}" use_sim="${use_sim}"/>
+</xacro:if>
+<xacro:if value="${tool == 'none'}">
+  <xacro:mod101_tool_none prefix="${prefix}" use_sim="${use_sim}"/>
+</xacro:if>
 </xacro:macro>
 </robot>

File: src/mod101_description/urdf/modules/shoulder_big.xacro (robot description, xacro)
@@ -3,11 +3,14 @@
   Shoulder joint module — BIG (ST3120). Same interface links/joints as
   shoulder_small.xacro, but the larger servo + heavier brackets from the
-  mod101_large export. The large export sits in a different CAD canvas, so the
-  three meshes are registered as ONE rigid unit: a single offset anchors the
-  module's input link (shoulder_rotation_link) exactly on the small one, which
-  preserves the servo<->bracket mating from the large export. Residual ~1 cm
-  from the exports' ~1.5° relative rotation — re-export the big parts in the
-  small frame (or send a same-frame mod101-big export) to zero it; then these
-  visual origins just become the export's own.
+  mod101_large export. The three meshes are registered as ONE rigid unit
+  (visual origins satisfy V_servo = V_rot - fixed_servo_shoulder and
+  V_adapter = V_servo - joint_shoulder, exactly as in the small module), so the
+  assembly moves together.
+  The big parts are now exported in the same CAD frame as the small ones, so
+  the visual origins below are the export's own and the nudge is zero: the
+  adapter's rail slot straddles the 20x20 extrusion axis to within ~1.5 mm and
+  the rotation link is centred on the joint_base axis to within ~1 mm — the
+  same fit the small module has. Don't re-introduce a nudge to "fix" apparent
+  offset; check the datums first (see below).
 -->
 <robot xmlns:xacro="http://www.ros.org/wiki/xacro">
@@ -15,9 +18,15 @@
 <!-- Fine-alignment nudge for the whole big-shoulder assembly (cosmetic; shifts
      all three meshes together, kinematics unchanged). Editable live from the
-     configurator's nudge panel, or by hand here. Zero out after a same-frame
-     re-export. -->
-<xacro:property name="snx" value="0.014000"/>
-<xacro:property name="sny" value="0.026500"/>
-<xacro:property name="snz" value="0.006000"/>
+     configurator's nudge panel, or by hand here.
+     Zero, and it should stay zero for this export. The datums to check if you
+     think it needs adjusting (all in link-local coords):
+       shoulder_adapter_1  AABB centre should sit on the arm_extrusion axis,
+                           i.e. (y,z) = (-0.019171, -0.001125)
+       shoulder_rotation_link_1  AABB should be centred on y=0 (the joint_base
+                           axis, which passes through the link origin)
+     A stale non-zero nudge here was displacing the whole assembly ~26 mm. -->
+<xacro:property name="snx" value="0.000000"/>
+<xacro:property name="sny" value="0.000000"/>
+<xacro:property name="snz" value="0.000000"/>
 <link name="${prefix}shoulder_rotation_link_1">
   <inertial>
