Commit message: moveit

File: src/mod101_control/urdf/mod101.hardware.xacro (robot description, xacro)
@@ -7,5 +7,8 @@
   servo bus driver once that lands.
 -->
-<robot name="mod101_hardware" xmlns:xacro="http://www.ros.org/wiki/xacro">
+<!-- NB: the robot name must stay "mod101" — it has to match the name in
+     mod101_moveit_config's SRDF, or MoveIt refuses to load with "semantic
+     description is not specified for the same robot as the URDF". -->
+<robot name="mod101" xmlns:xacro="http://www.ros.org/wiki/xacro">
   <xacro:arg name="use_sim" default="false"/>
   <xacro:include filename="$(find mod101_description)/urdf/mod101.xacro"/>

File: src/mod101_description/urdf/mod101.xacro (robot description, xacro)
@@ -12,16 +12,9 @@
      gazebo extensions. Hardware overlays (mod101_control) override to false. -->
 <xacro:arg name="use_sim" default="true"/>
-<!-- tool: which end-effector package to pull in. The arm terminates at
-     `wrist_flange`; the selected tool's URDF attaches its root link there and
-     contributes its own joints, ros2_control hardware block, gazebo extensions,
-     controllers, and (via the gazebo launch) its own launch fragment. Must
-     match a package `mod101_tool_<tool>` shipping urdf/tool.urdf.xacro.
-     The configurator reads/writes this default. -->
-<xacro:arg name="tool" default="pincopen"/>
-<!-- Build parameters: two rail lengths + two servo-mount variants (small|big). -->
-<xacro:arg name="shoulder_ext_length" default="0.0820"/>
-<xacro:arg name="elbow_ext_length"    default="0.0980"/>
-<xacro:arg name="shoulder_mount"      default="small"/>
-<xacro:arg name="elbow_mount"         default="small"/>
+<!-- tool + the four build args come from the configured-arm file, which the
+     web configurator owns. Do not redeclare them here: base101 (and anything
+     else that instantiates the macro) includes the same file, so a
+     configurator change reaches every consumer on the next build. -->
+<xacro:include filename="$(find mod101_description)/urdf/mod101_config.xacro" />
 <xacro:include filename="$(find mod101_description)/urdf/materials.xacro" />
 <xacro:include filename="$(find mod101_description)/urdf/mod101_macro.xacro" />

File: src/mod101_description/urdf/mod101_macro.xacro (robot description, xacro)
@@ -41,5 +41,5 @@
 <xacro:property name="ext_cross"         value="0.020"/>  <!-- 20x20 mm -->
 <xacro:property name="extrusion_density" value="0.46"/>   <!-- kg/m -->
-<xacro:macro name="mod101_arm" params="prefix:='' parent:='' xyz:='0 0 0' rpy:='0 0 0' tool:='jaws' use_sim:='true' shoulder_ext_length:='0.082' elbow_ext_length:='0.098' shoulder_mount:='small' elbow_mount:='small'">
+<xacro:macro name="mod101_arm" params="prefix:='' parent:='' xyz:='0 0 0' rpy:='0 0 0' tool:='jaws' use_sim:='true' shoulder_ext_length:=0.082 elbow_ext_length:=0.098 shoulder_mount:='small' elbow_mount:='small'">
 <!-- Rail length IS the joint advance along local X (1:1). The extrusion link is
      a box primitive of this length, so editing the length scales the rail AND
@@ -61,18 +61,25 @@
   </joint>
 </xacro:unless>
+<!-- base_link is re-centred on the base plate: origin at the centre of the
+     100x120 mm footprint, on the underside mounting face. The CAD export put
+     it ~1.4 cm/7.3 cm/6.4 cm off in the corner and below the plate, which made
+     every caller hand-tune its mount xyz. Callers can now bolt the arm down
+     with the plain deck-centre / deck-top offset. -->
 <link name="${prefix}base_link">
   <inertial>
-    <origin xyz="-0.016083210300696003 0.07326726540183791 0.07387020603487769" rpy="0 0 0"/>
-    <mass value="0.8668211242819505"/>
-    <inertia ixx="0.001015" iyy="0.000946" izz="0.001687" ixy="4e-06" iyz="-3e-06" ixz="0.000152"/>
-  </inertial>
-  <visual>
-    <origin xyz="0 0 0" rpy="0 0 0"/>
+    <origin xyz="-0.008702404 0.000111487 0.00989655" rpy="0 0 0"/>
+    <mass value="0.0832840557"/>
+    <inertia ixx="9.7521062e-05" iyy="9.08915514e-05" izz="0.000162086731" ixy="3.84319456e-07" iyz="-2.88239592e-07" ixz="1.46041393e-05"/>
+  </inertial>
+  <visual>
+    <origin xyz="0.007380806 -0.073155779 -0.063973656" rpy="0 0 0"/>
     <geometry><mesh filename="file://$(find mod101_description)/meshes/base_link.stl" scale="0.001 0.001 0.001"/></geometry>
     <material name="body_darkgrey"/>
   </visual>
   <collision>
-    <origin xyz="0 0 0" rpy="0 0 0"/>
-    <geometry><mesh filename="file://$(find mod101_description)/meshes/base_link.stl" scale="0.001 0.001 0.001"/></geometry>
+    <origin xyz="0 0 0.0265" rpy="0 0 0"/>
+    <geometry>
+      <box size="0.1 0.12 0.053"/>
+    </geometry>
   </collision>
 </link>
@@ -89,6 +96,8 @@
   </visual>
   <collision>
-    <origin xyz="0.033981 -0.084076 -0.113974" rpy="0 0 0"/>
-    <geometry><mesh filename="file://$(find mod101_description)/meshes/servo_base_1.stl" scale="0.001 0.001 0.001"/></geometry>
+    <origin xyz="0.0165002 -0.0102503 -0.0157003" rpy="0 0 0"/>
+    <geometry>
+      <box size="0.0452234 0.0247234 0.0378"/>
+    </geometry>
   </collision>
 </link>
@@ -96,6 +105,6 @@
   <inertial>
     <origin xyz="0.02230051687619229 0.01594291177721944 -3.4268786498758974e-07" rpy="0 0 0"/>
-    <mass value="0.1881374899503161"/>
-    <inertia ixx="6e-05" iyy="0.000108" izz="0.000142" ixy="1e-06" iyz="0.0" ixz="-0.0"/>
+    <mass value="0.0257291587"/>
+    <inertia ixx="8.20543276e-06" iyy="1.4769779e-05" izz="1.94195242e-05" ixy="1.36757213e-07" iyz="0" ixz="-0"/>
   </inertial>
   <visual>
@@ -105,6 +114,8 @@
   </visual>
   <collision>
-    <origin xyz="0.045885 -0.058276 -0.097774" rpy="0 0 0"/>
-    <geometry><mesh filename="file://$(find mod101_description)/meshes/base_cover_1.stl" scale="0.001 0.001 0.001"/></geometry>
+    <origin xyz="0.0202023 0.0158002 -3.45062e-07" rpy="0 0 0"/>
+    <geometry>
+      <box size="0.0684038 0.0395731 0.0286"/>
+    </geometry>
   </collision>
 </link>
@@ -170,6 +181,6 @@
   <inertial>
     <origin xyz="-0.0019161875719076876 -0.001239865018947961 -8.234763106684806e-07" rpy="0 0 0"/>
-    <mass value="0.1802416209536359"/>
-    <inertia ixx="5.5e-05" iyy="2.2e-05" izz="5.1e-05" ixy="1e-06" iyz="0.0" ixz="0.0"/>
+    <mass value="0.0198664172"/>
+    <inertia ixx="6.06215668e-06" iyy="2.42486267e-06" izz="5.62127255e-06" ixy="1.1022103e-07" iyz="0" ixz="0"/>
   </inertial>
   <visual>
@@ -179,6 +190,8 @@
   </visual>
   <collision>
-    <origin xyz="-0.035419 -0.074758 -0.173765" rpy="0 0 0"/>
-    <geometry><mesh filename="file://$(find mod101_description)/meshes/wrist_servo_adapter_1.stl" scale="0.001 0.001 0.001"/></geometry>
+    <origin xyz="0.000500196 -0.000549624 -2.37122e-07" rpy="0 0 0"/>
+    <geometry>
+      <box size="0.033 0.0493 0.0268"/>
+    </geometry>
   </collision>
 </link>
@@ -195,6 +208,8 @@
   </visual>
   <collision>
-    <origin xyz="-0.045069 -0.090758 -0.184015" rpy="0 0 0"/>
-    <geometry><mesh filename="file://$(find mod101_description)/meshes/servo_wrist_tilt_1.stl" scale="0.001 0.001 0.001"/></geometry>
+    <origin xyz="0.0202502 -0.0162996 -0.0102502" rpy="0 0 0"/>
+    <geometry>
+      <box size="0.0452234 0.0378 0.0247234"/>
+    </geometry>
   </collision>
 </link>
@@ -202,6 +217,6 @@
   <inertial>
     <origin xyz="0.0265390165786311 0.018652019649215763 0.02086935983869931" rpy="0 0 0"/>
-    <mass value="0.19133626761871975"/>
-    <inertia ixx="0.000113" iyy="0.000128" izz="9.2e-05" ixy="-0.0" iyz="0.0" ixz="-4.5e-05"/>
+    <mass value="0.0264696078"/>
+    <inertia ixx="1.56325077e-05" iyy="1.77076194e-05" izz="1.27273514e-05" ixy="-0" iyz="0" ixz="-6.22533494e-06"/>
   </inertial>
   <visual>
@@ -211,6 +226,8 @@
   </visual>
   <collision>
-    <origin xyz="-0.077819 -0.055558 -0.173765" rpy="0 0 0"/>
-    <geometry><mesh filename="file://$(find mod101_description)/meshes/wrist_roll_adapter_1.stl" scale="0.001 0.001 0.001"/></geometry>
+    <origin xyz="0.0256497 0.0186504 0.0177044" rpy="0 0 0"/>
+    <geometry>
+      <box size="0.073299 0.0493 0.0573908"/>
+    </geometry>
   </collision>
 </link>
@@ -227,6 +244,8 @@
   </visual>
   <collision>
-    <origin xyz="-0.137219 -0.084458 -0.202765" rpy="0 0 0"/>
-    <geometry><mesh filename="file://$(find mod101_description)/meshes/servo_wrist_rotation_1.stl" scale="0.001 0.001 0.001"/></geometry>
+    <origin xyz="-0.0156998 -0.0102496 -0.0165002" rpy="0 0 0"/>
+    <geometry>
+      <box size="0.0378 0.0247234 0.0452234"/>
+    </geometry>
   </collision>
 </link>
@@ -234,6 +253,6 @@
   <inertial>
     <origin xyz="-0.015133427944392153 -0.00999962387213657 0.00491529865458315" rpy="0 0 0"/>
-    <mass value="0.07287491005104513"/>
-    <inertia ixx="1.7e-05" iyy="1.4e-05" izz="2.7e-05" ixy="0.0" iyz="-0.0" ixz="-0.0"/>
+    <mass value="0.011514241"/>
+    <inertia ixx="2.68600122e-06" iyy="2.21200101e-06" izz="4.26600194e-06" ixy="0" iyz="-0" ixz="-0"/>
   </inertial>
   <visual>
@@ -243,6 +262,8 @@
   </visual>
   <collision>
-    <origin xyz="-0.135219 -0.084908 -0.220165" rpy="0 0 0"/>
-    <geometry><mesh filename="file://$(find mod101_description)/meshes/camera_adapter_1.stl" scale="0.001 0.001 0.001"/></geometry>
+    <origin xyz="-0.0140503 -0.00999963 0.00747259" rpy="0 0 0"/>
+    <geometry>
+      <box size="0.042699 0.0388 0.0210544"/>
+    </geometry>
   </collision>
 </link>
@@ -250,6 +271,6 @@
   <inertial>
     <origin xyz="0.14361888944153076 0.3347919124721062 -0.15696687867817244" rpy="0 0 0"/>
-    <mass value="0.06632884156356747"/>
-    <inertia ixx="2.7e-05" iyy="2.5e-05" izz="9e-06" ixy="0.0" iyz="-0.0" ixz="5e-06"/>
+    <mass value="0.0104777712"/>
+    <inertia ixx="4.26511024e-06" iyy="3.94917615e-06" izz="1.42170341e-06" ixy="0" iyz="-0" ixz="7.89835229e-07"/>
   </inertial>
   <visual>
@@ -259,6 +280,8 @@
   </visual>
   <collision>
-    <origin xyz="0.025688 0.259707 -0.40513" rpy="0 0 0"/>
-    <geometry><mesh filename="file://$(find mod101_description)/meshes/camera_wing_1.stl" scale="0.001 0.001 0.001"/></geometry>
+    <origin xyz="0.143097 0.334715 -0.148664" rpy="0 0 0"/>
+    <geometry>
+      <box size="0.0276196 0.031 0.0625861"/>
+    </geometry>
   </collision>
 </link>
@@ -266,6 +289,6 @@
   <inertial>
     <origin xyz="-0.005107415957823297 0.012044156369510242 -0.01085870058537286" rpy="0 0 0"/>
-    <mass value="0.016638125458728874"/>
-    <inertia ixx="1e-06" iyy="1e-06" izz="1e-06" ixy="-0.0" iyz="0.0" ixz="-0.0"/>
+    <mass value="0.0166"/>
+    <inertia ixx="9.97708548e-07" iyy="9.97708548e-07" izz="9.97708548e-07" ixy="-0" iyz="0" ixz="-0"/>
   </inertial>
   <visual>
@@ -275,6 +298,8 @@
   </visual>
   <collision>
-    <origin xyz="-0.115073 -0.062344 -0.284896" rpy="0 0 0"/>
-    <geometry><mesh filename="file://$(find mod101_description)/meshes/wrist_camera_v1_1.stl" scale="0.001 0.001 0.001"/></geometry>
+    <origin xyz="-0.00532676 0.0119999 -0.010453" rpy="0 0 0"/>
+    <geometry>
+      <box size="0.0149472 0.028 0.0262219"/>
+    </geometry>
   </collision>
 </link>
@@ -291,10 +316,10 @@
 <!-- ===================== joints (canonical names, export axes) ============== -->
 <joint name="${prefix}fixed_servo_base_1" type="fixed">
-  <origin xyz="-0.033981 0.084076 0.113974" rpy="0 0 0"/>
+  <origin xyz="-0.026600194 0.010920221 0.050000344" rpy="0 0 0"/>
   <parent link="${prefix}base_link"/>
   <child link="${prefix}servo_base_1"/>
 </joint>
 <joint name="${prefix}fixed_base_cover_1" type="fixed">
-  <origin xyz="-0.045885 0.058276 0.097774" rpy="0 0 0"/>
+  <origin xyz="-0.038504194 -0.014879779 0.033800344" rpy="0 0 0"/>
   <parent link="${prefix}base_link"/>
   <child link="${prefix}base_cover_1"/>

File: src/mod101_description/urdf/modules/elbow_big.xacro (robot description, xacro)
@@ -20,6 +20,6 @@
   <inertial>
     <origin xyz="-0.010386839428546318 0.00039485016823848085 -0.0020812304383783786" rpy="0 0 0"/>
-    <mass value="1.0939"/>
-    <inertia ixx="0.000337" iyy="0.000279" izz="0.000486" ixy="-6e-06" iyz="3e-06" ixz="-1e-05"/>
+    <mass value="0.0688074115"/>
+    <inertia ixx="2.11976393e-05" iyy="1.75493809e-05" izz="3.05698894e-05" ixy="-3.77406042e-07" iyz="1.88703021e-07" ixz="-6.2901007e-07"/>
   </inertial>
   <visual>
@@ -29,6 +29,8 @@
   </visual>
   <collision>
-    <origin xyz="${0.093660+enx} ${0.003135+eny} ${-0.065996+enz}" rpy="0 0 0"/>
-    <geometry><mesh filename="file://$(find mod101_description)/meshes/elbow_link_big_1.stl" scale="0.001 0.001 0.001"/></geometry>
+    <origin xyz="${(0.093660+enx) + -0.105036} ${(0.003135+eny) + -0.00124135} ${(-0.065996+enz) + 0.072475}" rpy="0 0 0"/>
+    <geometry>
+      <box size="0.0733383 0.0747 0.03655"/>
+    </geometry>
   </collision>
 </link>
@@ -45,6 +47,8 @@
   </visual>
   <collision>
-    <origin xyz="${0.128120+enx} ${0.018005+eny} ${-0.069671+enz}" rpy="0 0 0"/>
-    <geometry><mesh filename="file://$(find mod101_description)/meshes/servo_elbow_big_1.stl" scale="0.001 0.001 0.001"/></geometry>
+    <origin xyz="${(0.128120+enx) + -0.126455} ${(0.018005+eny) + -0.00124135} ${(-0.069671+enz) + 0.09075}" rpy="0 0 0"/>
+    <geometry>
+      <box size="0.03 0.0683 0.065"/>
+    </geometry>
   </collision>
 </link>
@@ -52,6 +56,6 @@
   <inertial>
     <origin xyz="0.020137826276852483 0.018502164445195313 0.00029332039965654366" rpy="0 0 0"/>
-    <mass value="0.4679"/>
-    <inertia ixx="0.000165" iyy="0.000101" izz="0.000213" ixy="0.0" iyz="-0.0" ixz="-2e-06"/>
+    <mass value="0.0407483489"/>
+    <inertia ixx="1.43694755e-05" iyy="8.79586074e-06" izz="1.85496865e-05" ixy="0" iyz="-0" ixz="-1.7417546e-07"/>
   </inertial>
   <visual>
@@ -61,6 +65,8 @@
   </visual>
   <collision>
-    <origin xyz="${0.117870+enx} ${0.021405+eny} ${-0.098671+enz}" rpy="0 0 0"/>
-    <geometry><mesh filename="file://$(find mod101_description)/meshes/elbow_adapter_big_1.stl" scale="0.001 0.001 0.001"/></geometry>
+    <origin xyz="${(0.117870+enx) + -0.104886} ${(0.021405+eny) + -0.00114134} ${(-0.098671+enz) + 0.10735}" rpy="0 0 0"/>
+    <geometry>
+      <box size="0.0730383 0.0747 0.0299"/>
+    </geometry>
   </collision>
 </link>

File: src/mod101_description/urdf/modules/elbow_small.xacro (robot description, xacro)
@@ -10,6 +10,6 @@
   <inertial>
     <origin xyz="-0.010386839428546318 0.00039485016823848085 -0.0020812304383783786" rpy="0 0 0"/>
-    <mass value="0.3445733336731394"/>
-    <inertia ixx="0.000106" iyy="8.8e-05" izz="0.000153" ixy="-2e-06" iyz="1e-06" ixz="-3e-06"/>
+    <mass value="0.0310526039"/>
+    <inertia ixx="9.55261389e-06" iyy="7.93047191e-06" izz="1.37882068e-05" ixy="-1.80237998e-07" iyz="9.01189989e-08" ixz="-2.70356997e-07"/>
   </inertial>
   <visual>
@@ -19,6 +19,8 @@
   </visual>
   <collision>
-    <origin xyz="0.062581 -0.073858 -0.142215" rpy="0 0 0"/>
-    <geometry><mesh filename="file://$(find mod101_description)/meshes/elbow_link_1.stl" scale="0.001 0.001 0.001"/></geometry>
+    <origin xyz="-0.0108048 0.000550375 0.00151226" rpy="0 0 0"/>
+    <geometry>
+      <box size="0.0536101 0.0493 0.029825"/>
+    </geometry>
   </collision>
 </link>
@@ -35,6 +37,8 @@
   </visual>
   <collision>
-    <origin xyz="0.097041 -0.058988 -0.14589" rpy="0 0 0"/>
-    <geometry><mesh filename="file://$(find mod101_description)/meshes/servo_elbow_1.stl" scale="0.001 0.001 0.001"/></geometry>
+    <origin xyz="0.0102501 0.0154997 0.0164998" rpy="0 0 0"/>
+    <geometry>
+      <box size="0.0247234 0.0378 0.0452234"/>
+    </geometry>
   </collision>
 </link>
@@ -42,6 +46,6 @@
   <inertial>
     <origin xyz="0.020137826276852483 0.018502164445195313 0.00029332039965654366" rpy="0 0 0"/>
-    <mass value="0.2129021996409237"/>
-    <inertia ixx="7.5e-05" iyy="4.6e-05" izz="9.7e-05" ixy="0.0" iyz="-0.0" ixz="-1e-06"/>
+    <mass value="0.0245465749"/>
+    <inertia ixx="8.64713056e-06" iyy="5.30357341e-06" izz="1.11836222e-05" ixy="0" iyz="-0" ixz="-1.15295074e-07"/>
   </inertial>
   <visual>
@@ -51,6 +55,8 @@
   </visual>
   <collision>
-    <origin xyz="0.086791 -0.055588 -0.17489" rpy="0 0 0"/>
-    <geometry><mesh filename="file://$(find mod101_description)/meshes/elbow_adapter_1.stl" scale="0.001 0.001 0.001"/></geometry>
+    <origin xyz="0.0132671 0.0186204 -2.29492e-07" rpy="0 0 0"/>
+    <geometry>
+      <box size="0.0538862 0.0493 0.0273769"/>
+    </geometry>
   </collision>
 </link>

File: src/mod101_description/urdf/modules/shoulder_big.xacro (robot description, xacro)
@@ -32,6 +32,6 @@
   <inertial>
     <origin xyz="0.032744272167771385 0.0004962194281389748 -0.013844865838515547" rpy="0 0 0"/>
-    <mass value="0.5298"/>
-    <inertia ixx="0.000197" iyy="0.00027" izz="0.000248" ixy="-3e-06" iyz="-2e-06" ixz="-2.5e-05"/>
+    <mass value="0.049583984"/>
+    <inertia ixx="1.84372307e-05" iyy="2.5269301e-05" izz="2.32103209e-05" ixy="-2.80770011e-07" iyz="-1.87180007e-07" ixz="-2.33975009e-06"/>
   </inertial>
   <visual>
@@ -41,6 +41,8 @@
   </visual>
   <collision>
-    <origin xyz="${-0.001130+snx} ${-0.000787+sny} ${-0.049192+snz}" rpy="0 0 0"/>
-    <geometry><mesh filename="file://$(find mod101_description)/meshes/shoulder_rotation_link_big_1.stl" scale="0.001 0.001 0.001"/></geometry>
+    <origin xyz="${(-0.001130+snx) + 0.0294865} ${(-0.000787+sny) + -0.000250002} ${(-0.049192+snz) + 0.03455}" rpy="0 0 0"/>
+    <geometry>
+      <box size="0.0809691 0.0747 0.0493"/>
+    </geometry>
   </collision>
 </link>
@@ -57,6 +59,8 @@
   </visual>
   <collision>
-    <origin xyz="${-0.059990+snx} ${0.015210+sny} ${-0.042608+snz}" rpy="0 0 0"/>
-    <geometry><mesh filename="file://$(find mod101_description)/meshes/servo_shoulder_big_1.stl" scale="0.001 0.001 0.001"/></geometry>
+    <origin xyz="${(-0.059990+snx) + 0.0547211} ${(0.015210+sny) + -0.000250002} ${(-0.042608+snz) + 0.0592}" rpy="0 0 0"/>
+    <geometry>
+      <box size="0.03 0.0683 0.065"/>
+    </geometry>
   </collision>
 </link>
@@ -64,6 +68,6 @@
   <inertial>
     <origin xyz="-0.020137432669050628 -0.01850241218843865 0.0002933203996578482" rpy="0 0 0"/>
-    <mass value="0.4682"/>
-    <inertia ixx="0.000165" iyy="0.000101" izz="0.000213" ixy="0.0" iyz="0.0" ixz="2e-06"/>
+    <mass value="0.0407909635"/>
+    <inertia ixx="1.43752861e-05" iyy="8.79941757e-06" izz="1.85571876e-05" ixy="0" iyz="0" ixz="1.74245893e-07"/>
   </inertial>
   <visual>
@@ -73,6 +77,8 @@
   </visual>
   <collision>
-    <origin xyz="${-0.049740+snx} ${-0.019990+sny} ${-0.075358+snz}" rpy="0 0 0"/>
-    <geometry><mesh filename="file://$(find mod101_description)/meshes/shoulder_adapter_big_1.stl" scale="0.001 0.001 0.001"/></geometry>
+    <origin xyz="${(-0.049740+snx) + 0.0331519} ${(-0.019990+sny) + -0.000150002} ${(-0.075358+snz) + 0.0758}" rpy="0 0 0"/>
+    <geometry>
+      <box size="0.0730383 0.0747 0.0299"/>
+    </geometry>
   </collision>
 </link>

File: src/mod101_description/urdf/modules/shoulder_small.xacro (robot description, xacro)
@@ -14,6 +14,6 @@
   <inertial>
     <origin xyz="0.032744272167771385 0.0004962194281389748 -0.013844865838515547" rpy="0 0 0"/>
-    <mass value="0.34166100376418634"/>
-    <inertia ixx="0.000127" iyy="0.000174" izz="0.00016" ixy="-2e-06" iyz="-1e-06" ixz="-1.6e-05"/>
+    <mass value="0.0329454964"/>
+    <inertia ixx="1.2246285e-05" iyy="1.67783748e-05" izz="1.54283906e-05" ixy="-1.92854883e-07" iyz="-9.64274413e-08" ixz="-1.54283906e-06"/>
   </inertial>
   <visual>
@@ -23,6 +23,8 @@
   </visual>
   <collision>
-    <origin xyz="0.004981 -0.073826 -0.117174" rpy="0 0 0"/>
-    <geometry><mesh filename="file://$(find mod101_description)/meshes/shoulder_rotation_link_1.stl" scale="0.001 0.001 0.001"/></geometry>
+    <origin xyz="0.024161 0.000578984 -0.0183751" rpy="0 0 0"/>
+    <geometry>
+      <box size="0.0756985 0.0493 0.0498091"/>
+    </geometry>
   </collision>
 </link>
@@ -39,6 +41,8 @@
   </visual>
   <collision>
-    <origin xyz="-0.053879 -0.057829 -0.11059" rpy="0 0 0"/>
-    <geometry><mesh filename="file://$(find mod101_description)/meshes/servo_shoulder_1.stl" scale="0.001 0.001 0.001"/></geometry>
+    <origin xyz="-0.0102497 0.0163 0.0202498" rpy="0 0 0"/>
+    <geometry>
+      <box size="0.0247234 0.0378 0.0452234"/>
+    </geometry>
   </collision>
 </link>
@@ -46,6 +50,6 @@
   <inertial>
     <origin xyz="-0.020137432669050628 -0.01850241218843865 0.0002933203996578482" rpy="0 0 0"/>
-    <mass value="0.2129021996409236"/>
-    <inertia ixx="7.5e-05" iyy="4.6e-05" izz="9.7e-05" ixy="0.0" iyz="0.0" ixz="1e-06"/>
+    <mass value="0.0245465762"/>
+    <inertia ixx="8.64713104e-06" iyy="5.3035737e-06" izz="1.11836228e-05" ixy="0" iyz="0" ixz="1.1529508e-07"/>
   </inertial>
   <visual>
@@ -55,6 +59,8 @@
   </visual>
   <collision>
-    <origin xyz="-0.043629 -0.093029 -0.14334" rpy="0 0 0"/>
-    <geometry><mesh filename="file://$(find mod101_description)/meshes/shoulder_adapter_1.stl" scale="0.001 0.001 0.001"/></geometry>
+    <origin xyz="-0.0132667 -0.0186206 -2.32544e-07" rpy="0 0 0"/>
+    <geometry>
+      <box size="0.0538862 0.0493 0.0273769"/>
+    </geometry>
   </collision>
 </link>

File: src/mod101_tool_jaws/urdf/tool.urdf.xacro (robot description, xacro)
@@ -58,6 +58,6 @@
     <inertial>
       <origin xyz="0.018214 -0.013763 -0.022966" rpy="0 0 0"/>
-      <mass value="0.447"/>
-      <inertia ixx="0.000264" iyy="0.000301" izz="0.000235" ixy="3.9e-05" iyz="-4e-05" ixz="8.2e-05"/>
+      <mass value="0.0437956016"/>
+      <inertia ixx="2.58658586e-05" iyy="2.94909979e-05" izz="2.30245333e-05" ixy="3.82109275e-06" iyz="-3.91906949e-06" ixz="8.03409246e-06"/>
     </inertial>
     <visual>
@@ -78,6 +78,6 @@
     <inertial>
       <origin xyz="-0.005824 -0.004501 -0.018111" rpy="0 0 0"/>
-      <mass value="0.284"/>
-      <inertia ixx="6.6e-05" iyy="4e-05" izz="6.9e-05" ixy="0.0" iyz="0.0" ixz="-6e-06"/>
+      <mass value="0.066"/>
+      <inertia ixx="1.53380282e-05" iyy="9.29577465e-06" izz="1.60352113e-05" ixy="0" iyz="0" ixz="-1.3943662e-06"/>
     </inertial>
     <visual>
@@ -98,6 +98,6 @@
     <inertial>
       <origin xyz="0.035386 -0.001620 -0.010188" rpy="0 0 0"/>
-      <mass value="0.159"/>
-      <inertia ixx="5.3e-05" iyy="8.7e-05" izz="4.1e-05" ixy="3e-06" iyz="-3e-06" ixz="2.3e-05"/>
+      <mass value="0.0180803214"/>
+      <inertia ixx="6.02677379e-06" iyy="9.89300604e-06" izz="4.66222124e-06" ixy="3.41138139e-07" iyz="-3.41138139e-07" ixz="2.6153924e-06"/>
     </inertial>
     <visual>
