Commit message: docker configuration, but it still sucks

File: src/mod101_harness/urdf/harness.gazebo.xacro (robot description, xacro)
@@ -8,8 +8,17 @@
 <robot xmlns:xacro="http://www.ros.org/wiki/xacro">
 <xacro:macro name="harness_gazebo" params="prefix:=''">
-  <xacro:property name="silver_color" value="Gazebo/Silver"/>
-  <xacro:macro name="hz_link" params="name">
+  <!-- The same three-way split the arm uses (mod101_description/urdf/
+       materials.xacro), not a second palette: extrusion is `silver`, every
+       bracket / adapter / camera body is dark grey, servo housings are black.
+       These Gazebo names have to track the URDF <material> on the same link —
+       the URDF colour is what RViz and the configurator's 3D preview draw, this
+       one is what Gazebo draws, and a mismatch means the robot looks like two
+       different robots depending on which window you are in. -->
+  <xacro:property name="silver_color"   value="Gazebo/Silver"/>
+  <xacro:property name="darkgrey_color" value="Gazebo/DarkGrey"/>
+  <xacro:property name="black_color"    value="Gazebo/Black"/>
+  <xacro:macro name="hz_link" params="name color">
     <gazebo reference="${prefix}${name}">
-      <material>${silver_color}</material>
+      <material>${color}</material>
       <mu1>0.2</mu1>
       <mu2>0.2</mu2>
@@ -17,4 +26,5 @@
     </gazebo>
   </xacro:macro>
+  <!-- 2020 extrusion: the base rail. -->
   <gazebo reference="${prefix}base_link">
     <material>${silver_color}</material>
@@ -24,12 +34,15 @@
     <gravity>true</gravity>
   </gazebo>
-  <xacro:hz_link name="yaw_bracket_1"/>
-  <xacro:hz_link name="yaw_servo_1"/>
-  <xacro:hz_link name="yaw_mount_1"/>
-  <xacro:hz_link name="pitch_servo_1"/>
-  <xacro:hz_link name="pitch_link__1"/>
-  <xacro:hz_link name="mod_101_adapter_1"/>
-  <xacro:hz_link name="tower_1"/>
-  <xacro:hz_link name="back_1"/>
+  <!-- extrusion -->
+  <xacro:hz_link name="tower_1"            color="${silver_color}"/>
+  <xacro:hz_link name="back_1"             color="${silver_color}"/>
+  <!-- brackets and adapters -->
+  <xacro:hz_link name="mod_101_adapter_1"  color="${darkgrey_color}"/>
+  <xacro:hz_link name="yaw_bracket_1"      color="${darkgrey_color}"/>
+  <xacro:hz_link name="yaw_mount_1"        color="${darkgrey_color}"/>
+  <xacro:hz_link name="pitch_link__1"      color="${darkgrey_color}"/>
+  <!-- servo housings -->
+  <xacro:hz_link name="yaw_servo_1"        color="${black_color}"/>
+  <xacro:hz_link name="pitch_servo_1"      color="${black_color}"/>
   <!-- Depth camera. rgbd_camera publishes color image, depth image, camera_info
        and a registered point cloud under <topic>. Stamp with the optical frame
@@ -38,5 +51,5 @@
        lens pointing along another axis, add a <pose> rotation on the sensor. -->
   <gazebo reference="${prefix}realsense_1">
-    <material>${silver_color}</material>
+    <material>${darkgrey_color}</material>
     <mu1>0.2</mu1>
     <mu2>0.2</mu2>

File: src/mod101_harness/urdf/harness_body.xacro (robot description, xacro)
@@ -18,5 +18,11 @@
     - removed the self-contained <xacro:include> of materials/gazebo/ros2control
     - `Revolute 18` -> `${prefix}pan_joint`, now `revolute` + limits
-    - `Revolute 20` -> `${prefix}tilt_joint`, now `revolute` + limits
+    - `Revolute 20` -> `${prefix}tilt_joint`, now `revolute` + limits, and its
+      AXIS CORRECTED from -X to +Y (see the joint for why)
+    - materials: the export painted every part `silver`. Now the harness reads
+      like the arm does, using the SAME palette (mod101_description/urdf/
+      materials.xacro) rather than a second one: `silver` for extrusion,
+      `body_darkgrey` for brackets/adapters/the camera body, `motor_black` for
+      servo housings.
     - added `${prefix}realsense_optical_frame` (REP-103 optical axes)
     - every link/joint name is `${prefix}`-scoped
@@ -55,5 +61,5 @@
       <mesh filename="file://$(find mod101_harness)/meshes/yaw_bracket_1.stl" scale="0.001 0.001 0.001"/>
     </geometry>
-    <material name="silver"/>
+    <material name="body_darkgrey"/>
   </visual>
   <collision>
@@ -75,5 +81,5 @@
       <mesh filename="file://$(find mod101_harness)/meshes/yaw_servo_1.stl" scale="0.001 0.001 0.001"/>
     </geometry>
-    <material name="silver"/>
+    <material name="motor_black"/>
   </visual>
   <collision>
@@ -95,5 +101,5 @@
       <mesh filename="file://$(find mod101_harness)/meshes/yaw_mount_1.stl" scale="0.001 0.001 0.001"/>
     </geometry>
-    <material name="silver"/>
+    <material name="body_darkgrey"/>
   </visual>
   <collision>
@@ -115,5 +121,5 @@
       <mesh filename="file://$(find mod101_harness)/meshes/pitch_servo_1.stl" scale="0.001 0.001 0.001"/>
     </geometry>
-    <material name="silver"/>
+    <material name="motor_black"/>
   </visual>
   <collision>
@@ -135,5 +141,5 @@
       <mesh filename="file://$(find mod101_harness)/meshes/pitch_link__1.stl" scale="0.001 0.001 0.001"/>
     </geometry>
-    <material name="silver"/>
+    <material name="body_darkgrey"/>
   </visual>
   <collision>
@@ -155,5 +161,5 @@
       <mesh filename="file://$(find mod101_harness)/meshes/realsense_1.stl" scale="0.001 0.001 0.001"/>
     </geometry>
-    <material name="silver"/>
+    <material name="body_darkgrey"/>
   </visual>
   <collision>
@@ -188,5 +194,5 @@
       <mesh filename="file://$(find mod101_harness)/meshes/mod_101_adapter_1.stl" scale="0.001 0.001 0.001"/>
     </geometry>
-    <material name="silver"/>
+    <material name="body_darkgrey"/>
   </visual>
   <collision>
@@ -262,10 +268,27 @@
   <child link="${prefix}pitch_servo_1"/>
 </joint>
-<!-- TILT (pitch). Was `continuous`; bounded like the pan joint. Axis -X. -->
+<!-- TILT (pitch). Was `continuous`; bounded like the pan joint.
+     AXIS CORRECTED, AND IT DISAGREES WITH THE CAD EXPORT. `Revolute 20` in
+     export/mod101_harness.raw.xacro has axis `-1 0 0`, which is the SAME
+     direction the camera looks: at pan=0 the RealSense boresight is +X, so a
+     rotation about X rolls the image and does not tilt it. Measured before the
+     change: sweeping pan over its full +-90 deg and tilt over its full +-80 deg,
+     the boresight pointed ABOVE THE HORIZON at every one of the 2929 sampled
+     pairs — the head could not be aimed at the table it is mounted over, or at
+     anything else below eye level.
+     A tilt axis has to be perpendicular to the boresight, so it is +Y. Positive
+     tilt now looks DOWN (rotating +X toward -Z), which is the aerospace pitch
+     sign and the one the pan/tilt group is commanded with.
+     THE CAD IS THE THING TO CHECK, NOT THIS LINE. Either the export's joint
+     axis is wrong or the RealSense body link is mounted a quarter turn off; the
+     mesh bounding boxes alone cannot tell which, because the pan servo and the
+     tilt servo have identical orientations in the export. If a re-export
+     changes this joint, re-run the boresight sweep in docs/harness-world.md
+     before trusting it. -->
 <joint name="${prefix}tilt_joint" type="revolute">
   <origin xyz="0.03405 -0.01025 0.029" rpy="0 0 0"/>
   <parent link="${prefix}pitch_servo_1"/>
   <child link="${prefix}pitch_link__1"/>
-  <axis xyz="-1.0 0.0 0.0"/>
+  <axis xyz="0.0 1.0 0.0"/>
   <limit lower="-1.396263" upper="1.396263" effort="5" velocity="3.0"/>
   <dynamics damping="0.05" friction="0.05"/>

Commit message: fixed motor ids in calibration and bug in harness

File: src/mod101_harness/urdf/harness.gazebo.xacro (robot description, xacro)
@@ -47,7 +47,13 @@
   <!-- Depth camera. rgbd_camera publishes color image, depth image, camera_info
        and a registered point cloud under <topic>. Stamp with the optical frame
-       so ROS consumers see REP-103 axes; the sensor still looks along
-       realsense_1 +X, which is where Gazebo aims it. If the viewer shows the
-       lens pointing along another axis, add a <pose> rotation on the sensor. -->
+       so ROS consumers see REP-103 axes.
+       THE <pose> IS LOAD-BEARING. Gazebo aims a camera sensor along its own +X
+       (with +Z up), and the sensor inherits the link frame unless posed. The
+       RealSense lens looks along realsense_1 -Y, not +X (see the optical-frame
+       note in harness_body.xacro for the mesh measurements), so without this
+       -90 deg yaw the simulated camera renders a view 90 deg off the real one,
+       while TF still says it points at -Y. The yaw maps sensor +X -> link -Y
+       and leaves sensor +Z on link +Z, so the image is upright and agrees with
+       ${prefix}realsense_optical_frame. -->
   <gazebo reference="${prefix}realsense_1">
     <material>${darkgrey_color}</material>
@@ -56,4 +62,5 @@
     <self_collide>true</self_collide>
     <sensor name="${prefix}depth_camera" type="rgbd_camera">
+      <pose>0 0 0 0 0 -1.570796</pose>
       <topic>harness/depth_camera</topic>
       <gz_frame_id>${prefix}realsense_optical_frame</gz_frame_id>

File: src/mod101_harness/urdf/harness_body.xacro (robot description, xacro)
@@ -18,6 +18,6 @@
     - removed the self-contained <xacro:include> of materials/gazebo/ros2control
     - `Revolute 18` -> `${prefix}pan_joint`, now `revolute` + limits
-    - `Revolute 20` -> `${prefix}tilt_joint`, now `revolute` + limits, and its
-      AXIS CORRECTED from -X to +Y (see the joint for why)
+    - `Revolute 20` -> `${prefix}tilt_joint`, now `revolute` + limits; axis kept
+      on the export's X, sign flipped to +X so positive tilt looks down
     - materials: the export painted every part `silver`. Now the harness reads
       like the arm does, using the SAME palette (mod101_description/urdf/
@@ -25,5 +25,6 @@
       `body_darkgrey` for brackets/adapters/the camera body, `motor_black` for
       servo housings.
-    - added `${prefix}realsense_optical_frame` (REP-103 optical axes)
+    - added `${prefix}realsense_optical_frame` (REP-103 optical axes, +Z along
+      the -Y boresight)
     - every link/joint name is `${prefix}`-scoped
 -->
@@ -171,13 +172,20 @@
 </link>
 <!-- Optical frame for the depth camera: REP-103 (+Z out of the lens, +X right,
-     +Y down). `realsense_1` is the body frame the export uses; Gazebo aims the
-     sensor along its +X. ROS image/pointcloud consumers assume the optical
-     convention, so the sensor stamps messages with this frame (see
-     harness.gazebo.xacro gz_frame_id). Same rotation the mod101 wrist camera
-     uses (mod101_macro.xacro). Zero translation — lens offset within the body
-     link not measured; fix here if metric accuracy is needed. -->
+     +Y down). The lens looks along realsense_1 -Y. Evidence, from the meshes:
+     realsense_1 is 89.8 x 25.1 x 25.0 mm - a D435, whose 90 mm dimension is the
+     stereo baseline, and it lies along X, so X cannot be the viewing axis. And
+     1313 mm^2 of the camera's +Y face is flat and coplanar with 1593 mm^2 of
+     pitch_link__1's -Y face at Y=-200.34, with the whole bracket behind that
+     plane: +Y is the bolted mounting face, so the lens faces -Y.
+     This frame therefore maps optical +Z -> -Y (forward), +Y -> -Z (down),
+     +X -> -X (right, with the camera upright: nothing in the chain carries a
+     roll, so link +Z is up). It previously used the arm wrist camera's rotation
+     (rpy -pi/2 0 -pi/2), which aims +Z along +X - 90 deg off, which is what
+     made the head look like it pointed the wrong way.
+     Zero translation - lens offset within the body link not measured; fix here
+     if metric accuracy is needed. -->
 <link name="${prefix}realsense_optical_frame"/>
 <joint name="${prefix}realsense_optical_joint" type="fixed">
-  <origin xyz="0 0 0" rpy="-1.570796 0 -1.570796"/>
+  <origin xyz="0 0 0" rpy="-1.570796 0 3.141593"/>
   <parent link="${prefix}realsense_1"/>
   <child link="${prefix}realsense_optical_frame"/>
@@ -269,26 +277,27 @@
 </joint>
 <!-- TILT (pitch). Was `continuous`; bounded like the pan joint.
-     AXIS CORRECTED, AND IT DISAGREES WITH THE CAD EXPORT. `Revolute 20` in
-     export/mod101_harness.raw.xacro has axis `-1 0 0`, which is the SAME
-     direction the camera looks: at pan=0 the RealSense boresight is +X, so a
-     rotation about X rolls the image and does not tilt it. Measured before the
-     change: sweeping pan over its full +-90 deg and tilt over its full +-80 deg,
-     the boresight pointed ABOVE THE HORIZON at every one of the 2929 sampled
-     pairs — the head could not be aimed at the table it is mounted over, or at
-     anything else below eye level.
-     A tilt axis has to be perpendicular to the boresight, so it is +Y. Positive
-     tilt now looks DOWN (rotating +X toward -Z), which is the aerospace pitch
-     sign and the one the pan/tilt group is commanded with.
-     THE CAD IS THE THING TO CHECK, NOT THIS LINE. Either the export's joint
-     axis is wrong or the RealSense body link is mounted a quarter turn off; the
-     mesh bounding boxes alone cannot tell which, because the pan servo and the
-     tilt servo have identical orientations in the export. If a re-export
-     changes this joint, re-run the boresight sweep in docs/harness-world.md
-     before trusting it. -->
+     AXIS IS X, WHICH IS WHAT THE CAD EXPORT SAID. An earlier edit here changed
+     it to +Y on the premise that the RealSense boresight is +X. That premise is
+     wrong, and +Y is the one axis that breaks this joint completely: the true
+     boresight is -Y (see the sensor note on realsense_1), so rotating about +Y
+     spins the camera about its own optical axis. Tilt was pure image ROLL — the
+     head could not be aimed up or down at all, at any commanded value.
+     Measured from the meshes, which settle it without a re-export. Both servos
+     are the same 45.22 x 24.72 x 37.80 part (identical STLs, rotated 90 deg),
+     and each joint origin lands exactly on that servo's output face, centred on
+     the other two axes:
+       pan_joint  is 0.00 mm from yaw_servo_1   Z-max  -> shaft along Z
+       tilt_joint is 0.55 mm from pitch_servo_1 X-max  -> shaft along X
+     A shaft is normal to the face it emerges from, so the tilt axis is X. It is
+     also perpendicular to the -Y boresight, as a pan/tilt requires; +Y was not.
+     SIGN is ours, not the CAD's: the export says `-1 0 0`, which would make
+     positive tilt look UP. Positive = DOWN is kept here (aerospace pitch, and
+     what the pan_tilt group and profiles/mod101_harness.yaml are commanded
+     with), so the axis is +X. Only the sign differs from the export. -->
 <joint name="${prefix}tilt_joint" type="revolute">
   <origin xyz="0.03405 -0.01025 0.029" rpy="0 0 0"/>
   <parent link="${prefix}pitch_servo_1"/>
   <child link="${prefix}pitch_link__1"/>
-  <axis xyz="0.0 1.0 0.0"/>
+  <axis xyz="1.0 0.0 0.0"/>
   <limit lower="-1.396263" upper="1.396263" effort="5" velocity="3.0"/>
   <dynamics damping="0.05" friction="0.05"/>
